File: battery_charger.kicad_sch (KiCad schematic)
At the start: 10 parts, among them J1 BAT, J1 USB_C_Receptacle

Commit message: 0
Parts:
- removed J1: BAT, Connector_JST:JST_EH_B2B-EH-A_1x02_P2.50mm_Vertical, symbol PCM_SL_Connectors:JST_02
- added Q?: FS8205A, SOT-23-6L_TCP, symbol FS8205A:FS8205A
- added U1: DW01A, Package_TO_SOT_SMD:SOT-23-6, symbol Battery_Management:DW01A
Connections:
- net +5V: now also D1.1 (K); no longer D1.2 (A)
- net GND: no longer C1.2
- net at J1.A4 (VBUS), J1.A9 (VBUS), J1.B4 (VBUS)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: now also D1.2 (A); no longer D1.1 (K)
Other:
- moved on the sheet: D1
Changed lines of the file:
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@@
+	(wire
+		(pts
+			(xy 38.1 21.59) (xy 41.91 21.59)
+		)
+		(stroke
+			(width 0)
+			(type default)
+		)
+	)
 	(wire
 		(pts
@@
 		(pts
 			(xy 170.18 73.66) (xy 158.75 73.66)
+		)
+		(stroke
+			(width 0)
+			(type default)
+		)
+	)
+	(wire
+		(pts
+			(xy 49.53 21.59) (xy 53.34 21.59)
 		)
 		(stroke
@@
 	)
 	(symbol
-		(lib_id "PCM_SL_Connectors:JST_02")
-		(at 171.45 96.52 270)
-		(unit 1)
-		(exclude_from_sim no)
-		(in_bom yes)
-		(on_board yes)
-		(dnp no)
-		(fields_autoplaced yes)
-		(property "Reference" "J1"
-			(at 175.26 95.2499 90)
-			(effects
-				(font
-					(size 1.27 1.27)
-				)
-				(justify left)
-			)
-		)
-		(property "Value" "BAT"
-			(at 175.26 97.7899 90)
-			(effects
-				(font
-					(size 1.27 1.27)
-				)
-				(justify left)
-			)
-		)
-		(property "Footprint" "Connector_JST:JST_EH_B2B-EH-A_1x02_P2.50mm_Vertical"
-			(at 177.8 96.52 0)
-			(effects
-				(font
-					(size 1.27 1.27)
-				)
-				(hide yes)
-			)
-		)
-		(property "Datasheet" ""
-			(at 177.8 96.52 0)
-			(effects
-				(font
-					(size 1.27 1.27)
-				)
-				(hide yes)
-			)
-		)
-		(property "Description" "JST Connector  2 pins"
-			(at 171.45 96.52 0)
-			(effects
-				(font
-					(size 1.27 1.27)
-				)
-				(hide yes)
-			)
-		)
-		(pin "2"
-		)
-		(pin "1"
-		)
-		(instances
-			(project ""
-				(path "/4bcf26b0-4035-4f01-b8ca-837e298bcb24"
-					(reference "J1")
-					(unit 1)
-				)
-			)
-		)
-	)
-	(symbol
 		(lib_id "power:GND")
 		(at 22.86 87.63 0)
@@
 	)
 	(symbol
+		(lib_id "FS8205A:FS8205A")
+		(at 170.18 100.33 0)
+		(unit 1)
+		(exclude_from_sim no)
+		(in_bom yes)
+		(on_board yes)
+		(dnp no)
+		(fields_autoplaced yes)
+		(property "Reference" "Q?"
+			(at 190.5 90.17 0)
+			(effects
+				(font
+					(size 1.524 1.524)
+				)
+			)
+		)
+		(property "Value" "FS8205A"
+			(at 190.5 92.71 0)
+			(effects
+				(font
+					(size 1.524 1.524)
+				)
+			)
+		)
+		(property "Footprint" "SOT-23-6L_TCP"
+			(at 170.18 100.33 0)
+			(effects
+				(font
+					(size 1.27 1.27)
+					(italic yes)
+				)
+				(hide yes)
+			)
+		)
+		(property "Datasheet" "FS8205A"
+			(at 170.18 100.33 0)
+			(effects
+				(font
+					(size 1.27 1.27)
+					(italic yes)
+				)
+				(hide yes)
+			)
+		)
+		(property "Description" ""
+			(at 170.18 100.33 0)
+			(effects
+				(font
+					(size 1.27 1.27)
+				)
+				(hide yes)
+			)
+		)
+		(pin "1"
+		)
+		(pin "3"
+		)
+		(pin "2"
+		)
+		(pin "4"
+		)
+		(pin "6"
+		)
+		(pin "5"
+		)
+		(instances
+			(project ""
+				(path "/4bcf26b0-4035-4f01-b8ca-837e298bcb24"
+					(reference "Q?")
+					(unit 1)
+				)
+			)
+		)
+	)
+	(symbol
 		(lib_id "Device:R")
 		(at 173.99 67.31 90)
@@
 	(symbol
 		(lib_id "Device:D_Schottky")
-		(at 41.91 21.59 0)
+		(at 45.72 21.59 180)
 		(unit 1)
 		(exclude_from_sim no)
@@
 		(fields_autoplaced yes)
 		(property "Reference" "D1"
-			(at 41.5925 15.24 0)
+			(at 46.0375 15.24 0)
 			(effects
 				(font
@@
 		)
 		(property "Value" "D_Schottky"
-			(at 41.5925 17.78 0)
+			(at 46.0375 17.78 0)
 			(effects
 				(font
@@
 		)
 		(property "Footprint" ""
-			(at 41.91 21.59 0)
+			(at 45.72 21.59 0)
 			(effects
 				(font
@@
 		)
 		(property "Datasheet" "~"
-			(at 41.91 21.59 0)
+			(at 45.72 21.59 0)
 			(effects
 				(font
@@
 		)
 		(property "Description" "Schottky diode"
-			(at 41.91 21.59 0)
+			(at 45.72 21.59 0)
 			(effects
 				(font
@@
 	)
 	(symbol
-		(lib_id "power:GND")
-		(at 158.75 86.36 270)
-		(unit 1)
-		(exclude_from_sim no)
-		(in_bom yes)
-		(on_board yes)
-		(dnp no)
-		(fields_autoplaced yes)
-		(property "Reference" "#PWR07"
-			(at 152.4 86.36 0)
-			(effects
-				(font
-					(size 1.27 1.27)
-				)
-				(hide yes)
-			)
-		)
-		(property "Value" "GND"
-			(at 154.94 86.3599 90)
-			(effects
-				(font
-					(size 1.27 1.27)
-				)
-				(justify right)
-			)
-		)
-		(property "Footprint" ""
-			(at 158.75 86.36 0)
-			(effects
-				(font
-					(size 1.27 1.27)
-				)
-				(hide yes)
-			)
-		)
-		(property "Datasheet" ""
-			(at 158.75 86.36 0)
-			(effects
-				(font
-					(size 1.27 1.27)
-				)
-				(hide yes)
-			)
-		)
-		(property "Description" "Power symbol creates a global label with name \"GND\" , ground"
-			(at 158.75 86.36 0)
-			(effects
-				(font
-					(size 1.27 1.27)
-				)
-				(hide yes)
-			)
-		)
-		(pin "1"
-		)
-		(instances
-			(project ""
-				(path "/4bcf26b0-4035-4f01-b8ca-837e298bcb24"
-					(reference "#PWR07")
-					(unit 1)
-				)
-			)
-		)
-	)
-	(symbol
 		(lib_id "power:+5V")
 		(at 107.95 76.2 90)
@@
 	)
 	(symbol
+		(lib_id "Battery_Management:DW01A")
+		(at 139.7 100.33 0)
+		(unit 1)
+		(exclude_from_sim no)
+		(in_bom yes)
+		(on_board yes)
+		(dnp no)
+		(fields_autoplaced yes)
+		(property "Reference" "U1"
+			(at 139.7 90.17 0)
+			(effects
+				(font
+					(size 1.27 1.27)
+				)
+			)
+		)
+		(property "Value" "DW01A"
+			(at 139.7 92.71 0)
+			(effects
+				(font
+					(size 1.27 1.27)
+				)
+			)
+		)
+		(property "Footprint" "Package_TO_SOT_SMD:SOT-23-6"
+			(at 139.7 100.33 0)
+			(effects
+				(font
+					(size 1.27 1.27)
+				)
+				(hide yes)
+			)
+		)
+		(property "Datasheet" "https://hmsemi.com/downfile/DW01A.PDF"
+			(at 139.7 100.33 0)
+			(effects
+				(font
+					(size 1.27 1.27)
+				)
+				(hide yes)
+			)
+		)
+		(property "Description" "Overcharge, overcurrent and overdischarge protection IC for single cell lithium-ion/polymer battery"
+			(at 139.954 98.806 0)
+			(effects
+				(font
+					(size 1.27 1.27)
+				)
+				(hide yes)
+			)
+		)
+		(pin "5"
+		)
+		(pin "6"
+		)
+		(pin "1"
+		)
+		(pin "2"
+		)
+		(pin "3"
+		)
+		(pin "4"
+		)
+		(instances
+			(project ""
+				(path "/4bcf26b0-4035-4f01-b8ca-837e298bcb24"
+					(reference "U1")
+					(unit 1)
+				)
+			)
+		)
+	)
+	(symbol
 		(lib_id "PCM_SparkFun-LED:LED")
 		(at 180.34 77.47 0)
@@
 	(symbol
 		(lib_id "power:+5V")
-		(at 45.72 21.59 270)
+		(at 53.34 21.59 270)
 		(unit 1)
 		(exclude_from_sim no)
@@
 		(fields_autoplaced yes)
 		(property "Reference" "#PWR02"
-			(at 41.91 21.59 0)
+			(at 49.53 21.59 0)
 			(effects
 				(font
@@
 		)
 		(property "Value" "+5V"
-			(at 49.53 21.5899 90)
+			(at 57.15 21.5899 90)
 			(effects
 				(font
@@
 		)
 		(property "Footprint" ""
-			(at 45.72 21.59 0)
+			(at 53.34 21.59 0)
 			(effects
 				(font
@@
 		)
 		(property "Datasheet" ""
-			(at 45.72 21.59 0)
+			(at 53.34 21.59 0)
 			(effects
 				(font
@@
 		)
 		(property "Description" "Power symbol creates a global label with name \"+5V\""
-			(at 45.72 21.59 0)
-			(effects
-				(font
+			(at 53.34 21.59 0)
+			(effects
+				(font

Commit message: foo
Parts:
- removed U1: DW01A, Package_TO_SOT_SMD:SOT-23-6, symbol Battery_Management:DW01A
- R1: value 1k -> 1.2k
Other:
- moved on the sheet: C1, LED1, LED2, Q?, R1, R2, R3, U?

Commit message: bar
Parts:
- removed Q?: FS8205A, SOT-23-6L_TCP, symbol FS8205A:FS8205A
- added C?: 100-470uF-50V, symbol Device:C_Polarized
- added C?: 200uF RV>10V, symbol Device:C_Polarized
- added D? (x2): D_Schottky, symbol Device:D_Schottky
- added J2, J?: JST_02, Connector_JST:JST_EH_B2B-EH-A_1x02_P2.50mm_Vertical, symbol PCM_SL_Connectors:JST_02
- added L?: 33uH, symbol Device:L
- added U2: DW01A, Package_TO_SOT_SMD:SOT-23-6, symbol Battery_Management:DW01A
- added U3: FS8205A, symbol Customs:FS8205A
- added U?: LM2596S-5, Package_TO_SOT_SMD:TO-263-5_TabPin3, symbol Regulator_Switching:LM2596S-5
- gave numbers to parts that had none: 1
Connections:
- net +5V: now also LED1.2 (A), LED2.2 (A), C?.1, L?.2
- net GND: now also C1.2, U1.1 (TEMP), C?.2, C?.2, D?.1 (K), J?.2, U3.3 (S2), U?.3 (GND), U?.5 (~{ON}/OFF); no longer LED1.2 (A), LED2.2 (A)
- net +BATT: now reaches C1.1, U1.5 (BAT)
- net +BATT: now also J2.1, U2.5 (VCC)
- new net: D?.2 (A), J?.1
- new net: C?.1, U?.1 (VIN)
- new net: D?.2 (A), L?.1, U?.2 (OUT)
- new net: U2.2 (CS), U3.2 (D1-D2)
- new net: U2.1 (OD), U3.5 (G1)
- new net: U2.3 (OC), U3.7 (G2)
- new net +12V_SOLAR: D?.1 (K)
- new net -BATT: J2.2, U2.6 (GND), U3.1 (S1)
Other:
- moved on the sheet: D1, LED1, LED2, R1, R2, R3, U1

Commit message: V2 added
Parts:
- removed U3: FS8205A, symbol Customs:FS8205A
- added C?: 10uF, symbol Device:C
- added C? (x2): 100uF, symbol Device:C
- added C? (x2): 22uF, symbol Device:C
- added D? (x3): D, symbol Device:D
- added L?: L, symbol Device:L
- added Q?: FS8205A, EasyEDA:SOT-23-6_L2.9-W1.6-P0.95-LS2.8-BR, symbol EasyEDA:FS8205A_C908265
- added R?: 3.2k, symbol Device:R
- added R?: 1k, symbol Device:R
- added U?: MT3608, Package_TO_SOT_SMD:SOT-23-6, symbol Regulator_Switching:MT3608
- added U?: TPS2121RUXR, RUX0012A, symbol TPS2121RUXR:TPS2121RUXR
- C?: value 200uF RV>10V -> 200uF >10V
Connections:
- net +5V: now also D?.2 (A), U?.4 (EN); no longer C?.1, L?.2, U1.4 (VCC)
- net +BATT: now also C?.1, L?.1, U?.5 (IN)
- net -BATT: now also Q?.1 (S1)
- net GND: now also C?.1, C?.2, C?.2, C?.2, C?.2, Q?.3 (S2), R?.2, U?.12 (GND), U?.2 (GND), U?.3 (CP2)
- net at D?.2 (A), L?.1, U?.2 (OUT): now also C?.1, L?.2, U1.4 (VCC), D?.1 (K), U?.2 (IN2), U?.6 (PR1)
- net at U2.2 (CS): now also Q?.2 (D1/D2)
- net at U2.1 (OD): now also Q?.6 (G1)
- net at U2.3 (OC): now also Q?.4 (G2)
- new net: C?.1, U?.1 (OUT), U?.8 (OUT)
- new net: C?.1, D?.1 (K), D?.2 (A), R?.1
- new net: R?.1, R?.2, U?.3 (FB)
- new net: D?.2 (A), L?.2, U?.1 (SW)
- new net: C?.1, U?.5 (OV1)
- new net: D?.1 (K), U?.7 (IN1)
- new net: C?.2, U?.4 (OV2)
