File: bcV2/bcV2.kicad_sch (KiCad schematic)
At the start: 0 parts

Commit message: V2 beta
Parts:
- added C? (x6): 22uF, symbol Device:C
- added C? (x2): 0.1uF, symbol Device:C
- added C?: 2.2nF, symbol Device:C
- added C?: 10nF, symbol Device:C
- added C?: 220pF, symbol Device:C
- added D? (x2): D_Schottky, symbol Device:D_Schottky
- added D? (x2): LED, PCM_SparkFun-LED:LED_0603_1608Metric, symbol PCM_SparkFun-LED:LED
- added J? (x2): JST_02, Connector_JST:JST_EH_B2B-EH-A_1x02_P2.50mm_Vertical, symbol PCM_SL_Connectors:JST_02
- added L?: 2.2uH, symbol Device:L
- added P?: USB_C_Plug, symbol Connector:USB_C_Plug
- added R?: 39k, symbol Device:R
- added R?: 100k, symbol Device:R
- added R?: 56.2k, symbol Device:R
- added R?: 1k, symbol Device:R
- added R?: 10k, symbol Device:R
- added R?: 44k, symbol Device:R
- added U?: CN3791, EasyEDA:SSOP-10_L4.9-W3.9-P1.00-LS6.0-BL, symbol EasyEDA:CN3791
- added U?: TPS61088RHLT, EasyEDA:VQFN-20_L4.6-W3.6-P0.50-BL, symbol EasyEDA:TPS61088RHLT
Connections:
- new net: C?.1, C?.1, R?.1, U?.14 (VOUT), U?.15 (VOUT), U?.16 (VOUT)
- new net: C?.1, R?.1
- new net: C?.1, R?.2, U?.18 (COMP)
- new net: C?.2, U?.1 (VCC), U?.2 (EN)
- new net: R?.2, U?.19 (ILIM)
- new net: R?.2, R?.2, U?.17 (FB)
- new net: D?.2 (A), D?.2 (A), R?.2
- new net: D?.1 (K), U?.3 (~{CHRG})
- new net: D?.1 (K), U?.4 (~{DONE})
- new net: D?.2 (A), J?.1
- new net: C?.2, L?.2, R?.1, U?.4 (SW), U?.5 (SW), U?.6 (SW), U?.7 (SW)
- new net: D?.2 (A), P?.A4 (VBUS), P?.A9 (VBUS), P?.B4 (VBUS), P?.B9 (VBUS)
- new net: C?.2, U?.10 (SS)
- new net: R?.2, U?.3 (FSW)
- new net: C?.1, U?.8 (BOOT)
- new net +12V_SOLAR: C?.1, D?.1 (K), D?.1 (K), U?.9 (VCC)
- new net +BATT: C?.1, C?.1, C?.1, J?.1, L?.1, U?.7 (BAT), U?.9 (VIN)
- new net GND: C?.1, C?.1, C?.2, C?.2, C?.2, C?.2, C?.2, C?.2, C?.2, C?.2, J?.2, J?.2, P?.A1 (GND), P?.A12 (GND), P?.B1 (GND), P?.B12 (GND), P?.S1 (SHIELD), R?.1, R?.1, R?.1, U?.13 (MODE), U?.2 (GND), U?.20 (AGND), U?.21 (PGND)

Commit message: v2 additions and fixes
Parts:
- added C?: 220nF, symbol Device:C
- added C?: 100nF, symbol Device:C
- added Q?: AO3401A, PCM_Package_TO_SOT_SMD_AKL:SOT-23, symbol PCM_Transistor_MOSFET_AKL:AO3401A
- added R?: 10k, symbol Device:R
- added R?: TC33X-2-104E, EasyEDA:RES-ADJ-SMD_TC33X-2-104E, symbol EasyEDA:TC33X-2-104E
- added R?: 56.2k, symbol Device:R
- added R?: 120, symbol Device:R
- added R?: 5.1k, symbol Device:R
- added R?: 100m, symbol Device:R
- R?: value 56.2k -> 562k
- R?: value 10k -> 100k
Connections:
- net +12V_SOLAR: now also Q?.2 (S); no longer C?.1, U?.9 (VCC)
- net +BATT: now also R?.1
- net GND: now also C?.1, C?.2, R?.2, R?.2
- net at U?.1 (VG): now also C?.1
- net at U?.10 (DRV): now also Q?.1 (G)
- net at U?.5 (COM): now also R?.2
- net at U?.6 (MPPT): now also R?.2
- net at U?.8 (CSP): now also R?.2
- net at D?.2 (A), J?.1: now also R?.1
- net at P?.A5 (CC): now also R?.1
- new net: R?.1, R?.3
- new net: R?.1, R?.2
- new net: C?.1, Q?.3 (D), U?.9 (VCC)
- new net: C?.2, R?.1
Other:
- moved on the sheet: C?, D?, R?, U?
